File: pcb/sp0256al2/psion-speech-sp0256al2/b.sch (KiCad schematic (older format))
At the start: 15 parts, among them U6 Regulator_Switching_MT3608

Commit message: Updates
Connections:
- net +5V_PSION renamed 5VUSB
Changed lines of the file:
@@
 Power supply for psion. This feeds into VB on the psion connector (if jumpers\nare set up that way). The Psion is then powered by a step-up conversion \nfrom the 5V of the USB connector.
 Text GLabel 1575 2375 0    50   Input ~ 0
-+5V_PSION
+5VUSB
 $Comp
 L Device:R_Small R?
