File: pcb/sp0256al2/psion-speech-sp0256al2/psion-speech-sp0256al2.kicad_pcb (KiCad board)
At the start: 2 copper layers, 60 parts, among them J1 Connector_USB_B_Micro, J2 Conn_01x02_Female, J3 Conn_02x08_Odd_Even, U1 SP0256AL2, U6 4024, U7 4024, U8 SST39SF020, U9 Regulator_Switching_MT3608

Commit message: Updates
Parts:
- removed J2: Conn_01x02_Female, Connector_PinHeader_2.54mm:PinHeader_1x02_P2.54mm_Vertical
- added J4: Conn_01x02_Female, Connector_PinHeader_2.54mm:PinHeader_1x02_P2.54mm_Vertical, F.Cu at (131.6, 118.6)
- added U2: 74LS368, Package_SO:SOIC-14_3.9x8.7mm_P1.27mm, B.Cu at (89.8, 117.2)
- added U3: PAM8302AAD, Package_SO:SO-8_5.3x6.2mm_P1.27mm, F.Cu at (116.4, 91.8)
- added U4: 4011, Package_SO:SOIC-14_3.9x8.7mm_P1.27mm, F.Cu at (125.9, 93.0)
- added Y1: 3.2768MHz, psion_org_2:crystal_um4s, F.Cu at (88.2, 102.8)
- U6, U7: moved to B.Cu
- moved R2 134.9 mm to (41.0, 96.9)
- moved R6 134.9 mm to (41.0, 99.8)
- moved C10 134.9 mm to (50.1, 93.9)
- moved C11 134.9 mm to (37.6, 90.3)
- moved C2 134.9 mm to (32.1, 96.9)
- moved C3 134.9 mm to (54.8, 89.7)
- moved C4 134.9 mm to (54.8, 92.7)
- moved C5 134.9 mm to (36.8, 93.9)
- moved C6 134.9 mm to (43.6, 90.3)
- moved C7 134.9 mm to (49.6, 90.3)
- moved C8 134.9 mm to (41.2, 93.9)
- moved C9 134.9 mm to (45.7, 93.9)
- moved R1 134.9 mm to (36.6, 96.9)
- moved R3 134.9 mm to (45.4, 96.9)
- moved R4 134.9 mm to (49.8, 96.9)
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Connections:
- FB2 pad 2: (no net) -> Net-(FB2-Pad2)
- FB3 pad 2: (no net) -> Net-(FB3-Pad2)
- J3 pad 12: (no net) -> SS
- R3 pad 1: Net-(C5-Pad1) -> (no net)
- R4 pad 2: (no net) -> Net-(R4-Pad2)
- R5 pad 1: (no net) -> Net-(R5-Pad1)
- R6 pad 1: (no net) -> Net-(R6-Pad1)
- U1 pad 20: (no net) -> ALD
- U1 pad 9: (no net) -> LRQ
Other:
- board outline added: 72 x 37 mm

Commit message: Updates
Parts:
- added J2: AudioJack2_Ground_Switch, psion_org_2:truconnect_stereo_audio_5_pin, F.Cu at (105.5, 106.3)
- C3, C5, D4, JP1, JP3, R1, R17, R2, R23, R24, R25, U4, Y1: moved to B.Cu
- RV1: footprint Resistor_SMD:R_0805_2012Metric -> Potentiometer_THT:Potentiometer_Bourns_3296W_Vertical
- moved R23 96.6 mm to (46.0, 108.0), turned to 90 degrees
- moved D4 84.2 mm to (48.0, 106.5), turned to 90 degrees
- moved R25 83.8 mm to (53.5, 106.0), turned to 270 degrees
- moved C23 82.4 mm to (46.5, 112.5), turned to 270 degrees
- moved C22 80.0 mm to (52.0, 106.0), turned to 270 degrees
- moved C24 79.8 mm to (56.0, 103.0), turned to 270 degrees
- moved R24 78.0 mm to (51.0, 106.0), turned to 90 degrees
- moved D5 77.8 mm to (62.6, 99.5)
- moved JP7 77.7 mm to (51.0, 128.0)
- moved R26 77.6 mm to (59.5, 101.5)
- moved JP5 74.2 mm to (47.0, 122.0)
- moved JP11 73.8 mm to (59.5, 99.5)
- moved C25 73.1 mm to (55.5, 126.5)
- moved JP10 72.0 mm to (52.0, 100.0), turned to 270 degrees
- moved JP4 70.0 mm to (41.0, 113.0)
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Connections:
- R3 pad 1: (no net) -> Net-(J2-PadSN)
Other:
- outline, holes or cut-outs redrawn

Commit message: Updates
Parts:
- C10, C11, C8, C9, FB3, R16, R18, R3, R5, R6, U3: moved to B.Cu
- moved R15 74.4 mm to (93.7, 129.0), turned to 90 degrees
- moved FB3 74.0 mm to (98.0, 122.7), turned to 270 degrees
- moved FB2 68.4 mm to (101.6, 119.1), turned to 270 degrees
- moved R19 65.5 mm to (98.8, 129.0), turned to 270 degrees
- moved C7 63.9 mm to (102.9, 109.2), turned to 180 degrees
- moved R6 61.7 mm to (104.6, 112.0), turned to 90 degrees
- moved C11 56.6 mm to (97.8, 118.1), turned to 270 degrees
- moved C8 56.1 mm to (94.5, 101.3)
- moved C6 55.5 mm to (102.9, 112.8)
- moved R20 54.5 mm to (96.3, 129.0), turned to 270 degrees
- moved C9 52.9 mm to (94.5, 98.8)
- moved R22 45.4 mm to (59.7, 127.0), turned to 90 degrees
- moved R18 45.1 mm to (98.3, 113.8), turned to 270 degrees
- moved R21 44.5 mm to (62.0, 127.0), turned to 90 degrees
- moved FB1 37.0 mm to (74.2, 104.6), turned to 180 degrees
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Routing:
- net SOE: track 0.00 -> 29.4 mm, vias 0 -> 1
Other:
- copper layers 2 -> 4

Commit message: Updates
Parts:
- removed JP7: 5V_to_logic, psion_org_2:SolderJumper-2_P1.3mm_Open_Pad0.8x0.8mm
- removed JP8: 5V_to_Psion, psion_org_2:SolderJumper-2_P1.3mm_Open_Pad0.8x0.8mm
- removed JP9: 5V_switched_to_Psion, psion_org_2:SolderJumper-2_P1.3mm_Open_Pad0.8x0.8mm
- D6: moved to B.Cu
- moved FB1 2.29 mm to (71.9, 104.6), turned to 0 degrees
- moved C4 1.70 mm to (66.8, 108.2)
- moved J4 0.83 mm to (89.9, 99.8)
- moved C7 0.76 mm to (102.9, 110.0)
- moved C11 0.51 mm to (97.3, 118.1)
- moved C6 0.51 mm to (102.9, 113.3)
- moved R23 0.28 mm to (45.7, 108.0)
- moved R18 0.25 mm to (98.0, 113.8)
- moved FB3 0.25 mm to (97.8, 122.7)
Connections:
- C10 pad 1: SVCC -> +5V_LOGIC
- C11 pad 1: SVCC -> +5V_LOGIC
- FB1 pad 1: (no net) -> 5VUSB
- J3 pad 13: SVCC -> +5V_LOGIC
- JP10 pad 1: +5V_PSION -> 5VUSB
- R4 pad 1: SVCC -> +5V_LOGIC
- U1 pad 19: SVCC -> +5V_LOGIC
- U1 pad 22: SVCC -> +5V_LOGIC
- U1 pad 23: SVCC -> +5V_LOGIC
- U1 pad 7: SVCC -> +5V_LOGIC
- U3 pad 6: SVCC -> +5V_LOGIC
- U4 pad 14: SVCC -> +5V_LOGIC
Routing:
- net +5V_LOGIC: track 0.00 -> 179.5 mm, vias 0 -> 8
- net +10V_PSION: track 0.00 -> 89.4 mm, vias 0 -> 6
- net SD2: track 0.00 -> 83.3 mm, vias 0 -> 7
- net GND: track 0.00 -> 80.5 mm, vias 0 -> 28
- net SD0: track 0.00 -> 76.8 mm, vias 0 -> 3
- net SD1: track 0.00 -> 75.7 mm, vias 0 -> 4
- net SD3: track 0.00 -> 74.6 mm, vias 0 -> 4
- net SCLK: track 0.00 -> 69.3 mm, vias 0 -> 4
- net SD7: track 0.00 -> 57.4 mm, vias 0 -> 3
- net SD4: track 0.00 -> 56.8 mm, vias 0 -> 3
- net SD5: track 0.00 -> 55.5 mm, vias 0 -> 1
- net SMR: track 0.00 -> 50.9 mm, vias 0 -> 5
- net A17: track 0.00 -> 39.0 mm, vias 0 -> 2
- net Net-(C6-Pad2): track 0.00 -> 36.8 mm, vias 0 -> 2
- net Net-(C5-Pad1): track 0.00 -> 36.3 mm, vias 0 -> 4
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- added copper zone on In2.Cu, net +5V_LOGIC
- added copper zone on In1.Cu, net GND
Other:
- board text added: "Psion Organiser II Speech Adapter Oct 2022 V1.0"
- board text added: "menadue@gmail.com"
