File: pcb/sp0256al2/psion-speech-sp0256al2/psion-speech-sp0256al2.kicad_pcb (KiCad board)
At the start: 4 copper layers, 72 x 37 mm, 62 parts, among them J1 Connector_USB_B_Micro, J2 AudioJack2_Ground_Switch, J3 Conn_02x08_Odd_Even, J4 Conn_01x02_Female, U1 SP0256AL2, U2 74LS368, U3 PAM8302AAD, U4 4011, U6 4024, U7 4024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

Commit message: Updates
Parts:
- removed U2: 74LS368, Package_SO:SOIC-14_3.9x8.7mm_P1.27mm
- added U5: 74LS368, Package_SO:SOIC-16_3.9x9.9mm_P1.27mm, B.Cu at (90.0, 118.4)
- moved J2 0.29 mm to (105.5, 106.0)
Connections:
- C10 pad 1: +5V_LOGIC -> Net-(C10-Pad1)
- C11 pad 1: +5V_LOGIC -> SVCC
- J3 pad 13: +5V_LOGIC -> SVCC
- JP1 pad 2: +5V_LOGIC -> SVCC
- JP3 pad 2: +5V_LOGIC -> SVCC
- JP5 pad 2: +5V_LOGIC -> SVCC
- R4 pad 1: +5V_LOGIC -> SVCC
- U1 pad 19: +5V_LOGIC -> SVCC
- U1 pad 22: +5V_LOGIC -> SVCC
- U1 pad 23: +5V_LOGIC -> SVCC
- U1 pad 7: +5V_LOGIC -> SVCC
- U3 pad 6: +5V_LOGIC -> SVCC
- U4 pad 14: +5V_LOGIC -> Net-(C10-Pad1)
- U4 pad 3: (no net) -> SEL_SOE_0
- U6 pad 14: +5V_LOGIC -> SVCC
- U7 pad 14: +5V_LOGIC -> SVCC
- U8 pad 1: +5V_LOGIC -> SVCC
- U8 pad 22: (no net) -> SEL_SOE_0
- U8 pad 31: +5V_LOGIC -> SVCC
- U8 pad 32: +5V_LOGIC -> SVCC
Routing:
- net +5V_LOGIC: track 179.5 -> 0.00 mm, vias 8 -> 0
- net SVCC: track 0.00 -> 50.7 mm, vias 0 -> 8
- net GND: track 80.5 -> 97.2 mm
- net SEL_SOE_0: track 0.00 -> 16.0 mm, vias 0 -> 1
- net Net-(U7-Pad12): track 28.1 -> 12.2 mm, vias 3 -> 2
- net Net-(C10-Pad1): track 0.00 -> 12.5 mm, vias 0 -> 2
- net SEL_SOE_1: track 18.2 -> 26.3 mm, vias 2 -> 4
- net SD3: track 74.6 -> 68.9 mm, vias 4 -> 5
- net NOT_SEL_SOE_1: track 18.5 -> 22.2 mm, vias 2 -> 3
- net SD7: track 57.4 -> 59.2 mm
- net LRQ: track 10.6 -> 12.4 mm
- net N_SS: track 26.6 -> 28.2 mm
- net Net-(U5-Pad12): track 0.00 -> 1.27 mm
- net Net-(U2-Pad12): track 1.27 -> 0.00 mm
- net Net-(C9-Pad1): track 33.0 -> 32.0 mm
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- added copper zone on In2.Cu, net GND
- added copper zone on In1.Cu, net SVCC
- removed copper zone on In2.Cu, net +5V_LOGIC
- removed copper zone on In1.Cu, net GND
Other:
- board text added: "Psion Organiser II Speech Adapter Oct 2022 V1.1"
- board text removed: "Psion Organiser II Speech Adapter Oct 2022 V1.0"

Commit message: Updates
Parts:
- added R7: 47k, Resistor_SMD:R_0805_2012Metric, F.Cu at (63.2, 108.2)
Connections:
- C10 pad 1: Net-(C10-Pad1) -> SVCC
- U1 pad 22: SVCC -> GND
- U4 pad 14: Net-(C10-Pad1) -> SVCC
- U4 pad 3: SEL_SOE_0 -> (no net)
- U5 pad 1: (no net) -> GND
- U8 pad 22: SEL_SOE_0 -> N_SS
Routing:
- net SVCC: track 50.7 -> 67.2 mm, vias 8 -> 11
- net N_SS: track 28.2 -> 44.5 mm, vias 4 -> 5
- net SEL_SOE_0: track 16.0 -> 0.00 mm, vias 1 -> 0
- net Net-(C10-Pad1): track 12.5 -> 0.00 mm, vias 2 -> 0
- net SD5: track 55.5 -> 63.5 mm, vias 1 -> 3
- net GND: track 97.2 -> 101.5 mm, vias 28 -> 29
- net Net-(U7-Pad5): track 23.5 -> 22.2 mm
- net SD1: track 75.7 -> 76.8 mm
- net SMR: track 51.5 -> 52.4 mm

Commit message: Updates
Parts:
- added C12: 100nF, Capacitor_SMD:C_0805_2012Metric, F.Cu at (104.1, 122.9)
- added C13: nopop, Capacitor_SMD:C_1210_3225Metric_Pad1.33x2.70mm_HandSolder, B.Cu at (104.0, 100.5)
- added C14: 20uF, Capacitor_SMD:C_1210_3225Metric_Pad1.33x2.70mm_HandSolder, B.Cu at (107.8, 117.6)
- added C15: 20uF, Capacitor_SMD:C_1210_3225Metric_Pad1.33x2.70mm_HandSolder, B.Cu at (107.8, 122.8)
- added C16: 20uF, Capacitor_SMD:C_1210_3225Metric_Pad1.33x2.70mm_HandSolder, F.Cu at (77.5, 105.5)
- added R10: 47k, Resistor_SMD:R_0805_2012Metric, F.Cu at (87.4, 129.0)
- added R8: R_Small, Resistor_SMD:R_0805_2012Metric, F.Cu at (93.3, 99.2)
- added R9: R_Small, Resistor_SMD:R_0805_2012Metric, F.Cu at (93.3, 101.5)
- moved J4 0.72 mm to (89.2, 99.8)
Connections:
- C8 pad 1: Net-(C8-Pad1) -> Net-(C13-Pad2)
- C9 pad 1: Net-(C9-Pad1) -> Net-(C13-Pad1)
- FB2 pad 1: Net-(C9-Pad1) -> Net-(C13-Pad1)
- FB3 pad 1: Net-(C8-Pad1) -> Net-(C13-Pad2)
- J4 pad 1: Net-(C9-Pad1) -> Net-(J4-Pad1)
- J4 pad 2: Net-(C8-Pad1) -> Net-(J4-Pad2)
- U8 pad 22: N_SS -> SS
Routing:
- net Net-(C13-Pad2): track 0.00 -> 33.0 mm, vias 0 -> 3
- net Net-(C13-Pad1): track 0.00 -> 32.7 mm, vias 0 -> 2
- net Net-(C9-Pad1): track 32.0 -> 0.00 mm, vias 1 -> 0
- net Net-(C8-Pad1): track 29.6 -> 0.00 mm, vias 2 -> 0
- net SS: track 27.3 -> 52.5 mm, vias 1 -> 4
- net GND: track 101.5 -> 125.7 mm
- net SVCC: track 67.2 -> 89.6 mm
- net N_SS: track 44.5 -> 26.9 mm, vias 5 -> 4
- net Net-(C12-Pad1): track 6.70 -> 14.6 mm
- net Net-(J4-Pad2): track 0.00 -> 3.54 mm
- net Net-(J4-Pad1): track 0.00 -> 3.45 mm
Other:
- board text added: "Psion Organiser II Speech Adapter Nov 2022 V1.1"
- board text removed: "Psion Organiser II Speech Adapter Oct 2022 V1.1"

Commit message: Updates
Parts:
- R8, R9: moved to B.Cu
- moved R9 1.97 mm to (91.6, 102.6), turned to 270 degrees
- moved R8 1.66 mm to (91.6, 99.1), turned to 270 degrees
- moved J4 0.45 mm to (88.8, 99.6)
Routing:
- net Net-(C5-Pad1): track 37.0 -> 34.2 mm, vias 4 -> 5
- net Net-(C13-Pad1): track 32.7 -> 34.3 mm, vias 2 -> 1
- net Net-(C13-Pad2): track 33.0 -> 34.2 mm, vias 3 -> 2
- net Net-(J4-Pad1): track 3.45 -> 4.49 mm
Other:
- board text added: "Psion Organiser II Speech Adapter Dec 2022 V1.1"
- board text removed: "Psion Organiser II Speech Adapter Nov 2022 V1.1"
