File: pcb/sp0256al2/psion-speech-sp0256al2/_autosave-psion-speech-sp0256al2.sch (KiCad schematic (older format))
At the start: 30 parts, among them J1 Connector_USB_B_Micro, J2 AudioJack2_Ground_Switch, J3 Conn_02x08_Odd_Even, J4 Conn_01x02_Female, U1 SP0256AL2, U2 74LS368, U3 PAM8302AAD, U4 4011, Y1 3.2768MHz

Commit message: Updates
Parts:
- removed U2: 74LS368, Package_SO:SOIC-14_3.9x8.7mm_P1.27mm, symbol 74xx_IEEE:74LS368
- added U5: 74LS368, Package_SO:SOIC-16_3.9x9.9mm_P1.27mm, symbol 74xx:74LS368
Connections:
- net GND: now also U5.8 (GND)
- net LRQ: now also U5.14 (I6)
- net NOT_SEL_SOE_1: now also U5.9 (O4a)
- net N_SOE: now also U5.7 (O3a)
- net N_SS: now also U5.3 (O1a)
- net SD7: now also U5.11 (O5b)
- net SEL_SOE_1: now also U5.10 (I4), U5.15 (OEb)
- net SOE: now also U5.6 (I3)
- net SS: now also U5.2 (I1)
- net SVCC: now also U5.16 (VCC); no longer C10.1, U4.14 (VDD)
- new net: C10.1, U4.14 (VDD)
- new net: U5.12 (I5), U5.13 (O6b)
Changed lines of the file:
@@
 	2225 5350 2225 6225
 $Sheet
-S 5450 5700 1200 625
+S 3625 5250 1200 625
 U 6340FD7B
 F0 "Psion ROM" 50
@@
 Text GLabel 1875 2875 0    50   Input ~ 0
 SD5
-$Comp
-L 74xx_IEEE:74LS368 U2
-U 1 1 63421380
-P 6450 4050
-F 0 "U2" H 6450 4616 50  0000 C CNN
-F 1 "74LS368" H 6450 4525 50  0000 C CNN
-F 2 "Package_SO:SOIC-14_3.9x8.7mm_P1.27mm" H 6450 4050 50  0001 C CNN
-F 3 "" H 6450 4050 50  0001 C CNN
-	1    6450 4050
-	1    0    0    -1
-$EndComp
-Text GLabel 7000 4650 2    50   Input ~ 0
+Text GLabel 8450 5225 2    50   Input ~ 0
 SD7
-Wire Wire Line
-	5900 4650 5625 4650
-Wire Wire Line
-	5625 4650 5625 4950
-Wire Wire Line
-	5625 4950 7000 4950
-Wire Wire Line
-	7000 4950 7000 4750
-Text GLabel 5900 4750 0    50   Input ~ 0
+Text GLabel 7450 5325 0    50   Input ~ 0
 LRQ
-$Comp
-L power:GND #PWR08
-U 1 1 634277F0
-P 5400 3800
-F 0 "#PWR08" H 5400 3550 50  0001 C CNN
-F 1 "GND" H 5405 3627 50  0000 C CNN
-F 2 "" H 5400 3800 50  0001 C CNN
-F 3 "" H 5400 3800 50  0001 C CNN
-	1    5400 3800
-	-1   0    0    -1
-$EndComp
-Wire Wire Line
-	5900 3800 5400 3800
-Text GLabel 5900 3950 0    50   Input ~ 0
+Text GLabel 7450 4825 0    50   Input ~ 0
 SS
-Text GLabel 5900 4150 0    50   Input ~ 0
+Text GLabel 7450 5025 0    50   Input ~ 0
 SOE
-Text GLabel 7000 3950 2    50   Input ~ 0
+Text GLabel 8450 4825 2    50   Input ~ 0
 N_SS
-Text GLabel 7000 4150 2    50   Input ~ 0
+Text GLabel 8450 5025 2    50   Input ~ 0
 N_SOE
-Text GLabel 10350 5200 2    50   Input ~ 0
+Text GLabel 8100 4150 2    50   Input ~ 0
 SVCC
 Wire Wire Line
@@
 Wire Wire Line
 	9575 4825 9875 4825
-Text GLabel 5900 4250 0    50   Input ~ 0
+Text GLabel 6850 5125 0    50   Input ~ 0
 SEL_SOE_1
-Text GLabel 7000 4250 2    50   Input ~ 0
+Text GLabel 8450 5125 2    50   Input ~ 0
 NOT_SEL_SOE_1
 Text GLabel 10475 4725 2    50   Input ~ 0
@@
 	1    0    0    -1
 $EndComp
-Wire Wire Line
-	6450 3700 6600 3700
+$Comp
+L 74xx:74LS368 U5
+U 1 1 6360F2CE
+P 7950 5225
+F 0 "U5" H 8250 6100 50  0000 C CNN
+F 1 "74LS368" H 8375 6025 50  0000 C CNN
+F 2 "Package_SO:SOIC-16_3.9x9.9mm_P1.27mm" H 7950 5225 50  0001 C CNN
+F 3 "http://www.ti.com/lit/gpn/sn74LS368" H 7950 5225 50  0001 C CNN
+	1    7950 5225
+	1    0    0    -1
+$EndComp
+Wire Wire Line
+	8450 5325 8725 5325
+Wire Wire Line
+	8725 5325 8725 6425
+Wire Wire Line
+	8725 6425 7050 6425
+Wire Wire Line
+	7050 6425 7050 5225
+Wire Wire Line
+	7050 5225 7450 5225
+$Comp
+L power:GND #PWR0103
+U 1 1 6361864B
+P 7950 6075
+F 0 "#PWR0103" H 7950 5825 50  0001 C CNN
+F 1 "GND" H 7955 5902 50  0000 C CNN
+F 2 "" H 7950 6075 50  0001 C CNN
+F 3 "" H 7950 6075 50  0001 C CNN
+	1    7950 6075
+	1    0    0    -1
+$EndComp
+Wire Wire Line
+	7950 6075 7950 5925
+Wire Wire Line
+	7950 4150 8100 4150
+Wire Wire Line
+	7950 4150 7950 4525
+Wire Wire Line
+	7450 5125 7150 5125
+Wire Wire Line
+	7150 5625 7450 5625
+Wire Wire Line
+	7150 5125 7150 5625
+Connection ~ 7150 5125
+Wire Wire Line
+	7150 5125 6850 5125
 $EndSCHEMATC
