File: pcb/sp0256al2/psion-speech-sp0256al2/a.sch (KiCad schematic (older format))
At the start: 20 parts, among them U2 4024, U3 4024, U4 SST39SF020

Commit message: Updates
Parts:
- removed JP7: 5V_to_logic, psion_org_2:SolderJumper-2_P1.3mm_Open_Pad0.8x0.8mm, symbol Device:Jumper_NO_Small
- removed JP8: 5V_to_Psion, psion_org_2:SolderJumper-2_P1.3mm_Open_Pad0.8x0.8mm, symbol Device:Jumper_NO_Small
- removed JP9: 5V_switched_to_Psion, psion_org_2:SolderJumper-2_P1.3mm_Open_Pad0.8x0.8mm, symbol Device:Jumper_NO_Small
Changed lines of the file:
@@
 Text GLabel 9950 3825 2    50   Input ~ 0
 +5V_LOGIC
-Text GLabel 7400 4450 0    50   Input ~ 0
-+5V
-Text GLabel 7400 4750 0    50   Input ~ 0
-+5V_SWITCHED
-Text GLabel 9975 4450 2    50   Input ~ 0
-+5V_PSION
-$Comp
-L Device:Jumper_NO_Small JP7
-U 1 1 62F07812
-P 8200 3825
-F 0 "JP7" H 8200 3900 50  0000 C CNN
-F 1 "5V_to_logic" H 8200 3750 50  0000 C CNN
-F 2 "psion_org_2:SolderJumper-2_P1.3mm_Open_Pad0.8x0.8mm" H 8200 3825 50  0001 C CNN
-F 3 "~" H 8200 3825 50  0001 C CNN
-	1    8200 3825
-	1    0    0    -1
-$EndComp
-$Comp
-L Device:Jumper_NO_Small JP8
-U 1 1 62F0854D
-P 8200 4450
-F 0 "JP8" H 8200 4525 50  0000 C CNN
-F 1 "5V_to_Psion" H 8225 4375 50  0000 C CNN
-F 2 "psion_org_2:SolderJumper-2_P1.3mm_Open_Pad0.8x0.8mm" H 8200 4450 50  0001 C CNN
-F 3 "~" H 8200 4450 50  0001 C CNN
-	1    8200 4450
-	1    0    0    -1
-$EndComp
-$Comp
-L Device:Jumper_NO_Small JP9
-U 1 1 62F087A5
-P 8225 4750
-F 0 "JP9" H 8200 4825 50  0000 C CNN
-F 1 "5V_switched_to_Psion" H 8200 4650 50  0000 C CNN
-F 2 "psion_org_2:SolderJumper-2_P1.3mm_Open_Pad0.8x0.8mm" H 8225 4750 50  0001 C CNN
-F 3 "~" H 8225 4750 50  0001 C CNN
-	1    8225 4750
-	1    0    0    -1
-$EndComp
-Wire Wire Line
-	7800 3825 8100 3825
-Wire Wire Line
-	9975 4450 8675 4450
-Wire Wire Line
-	8325 4750 8675 4750
-Wire Wire Line
-	8675 4750 8675 4450
-Connection ~ 8675 4450
-Wire Wire Line
-	8675 4450 8300 4450
 Text GLabel 3950 3425 0    50   Input ~ 0
 +5V_LOGIC
@@
 	1    0    0    -1
 $EndComp
-Wire Wire Line
-	7400 4450 8100 4450
-Wire Wire Line
-	8300 3825 9950 3825
 Text GLabel 7800 3825 0    50   Input ~ 0
 SVCC
-Wire Wire Line
-	7400 4750 8125 4750
 Text GLabel 3675 3225 0    50   Input ~ 0
 +5V_LOGIC
 Wire Wire Line
 	3950 3225 3675 3225
+Wire Wire Line
+	7800 3825 9950 3825
 $EndSCHEMATC

Commit message: Updates
Connections:
- net ROMCE renamed SEL_SOE_0
Changed lines of the file:
@@
 	4550 3900 4550 3825
 Text GLabel 4350 775  0    50   Input ~ 0
-+5V_LOGIC
+SVCC
 Wire Wire Line
 	4550 1325 4550 775
 Wire Wire Line
 	4550 775  4350 775
-Text GLabel 9950 3825 2    50   Input ~ 0
-+5V_LOGIC
 Text GLabel 3950 3425 0    50   Input ~ 0
-+5V_LOGIC
-Text GLabel 3950 3725 0    50   Input ~ 0
-SOE
+SVCC
 Wire Wire Line
 	8025 1425 5800 1425
@@
 $EndComp
 Text GLabel 1950 1225 0    50   Input ~ 0
-+5V_LOGIC
+SVCC
 Text GLabel 1100 2400 0    50   Input ~ 0
-+5V_LOGIC
+SVCC
 Wire Wire Line
 	2150 1225 2150 1475
@@
 Wire Wire Line
 	2700 2500 2900 2500
-Text GLabel 3950 3625 0    50   Input ~ 0
-ROMCE
 Wire Wire Line
 	1950 1225 2150 1225
@@
 	8900 5100 9100 5100
 Text GLabel 9100 5100 2    50   Input ~ 0
-+5V_LOGIC
+SVCC
 Connection ~ 8900 5400
 Wire Wire Line
@@
 	1    0    0    -1
 $EndComp
-Text GLabel 7800 3825 0    50   Input ~ 0
-SVCC
 Text GLabel 3675 3225 0    50   Input ~ 0
-+5V_LOGIC
+SVCC
 Wire Wire Line
 	3950 3225 3675 3225
-Wire Wire Line
-	7800 3825 9950 3825
+Text GLabel 3950 3725 0    50   Input ~ 0
+SOE
+Text GLabel 3950 3625 0    50   Input ~ 0
+SEL_SOE_0
 $EndSCHEMATC

Commit message: Updates
Connections:
- net SEL_SOE_0 renamed N_SS
Changed lines of the file:
@@
 SOE
 Text GLabel 3950 3625 0    50   Input ~ 0
-SEL_SOE_0
+N_SS
 $EndSCHEMATC

Commit message: Updates
Parts:
- added R10: 47k, Resistor_SMD:R_0805_2012Metric, symbol Device:R_Small
Connections:
- net VCC: now also R10.1
- net N_SS renamed SS
- net SS: now also R10.2
Changed lines of the file:
@@
 SOE
 Text GLabel 3950 3625 0    50   Input ~ 0
-N_SS
+SS
+$Comp
+L Device:R_Small R10
+U 1 1 637B85F8
+P 6775 3575
+F 0 "R10" H 6834 3621 50  0000 L CNN
+F 1 "47k" H 6834 3530 50  0000 L CNN
+F 2 "Resistor_SMD:R_0805_2012Metric" H 6775 3575 50  0001 C CNN
+F 3 "~" H 6775 3575 50  0001 C CNN
+	1    6775 3575
+	1    0    0    -1
+$EndComp
+Text GLabel 6675 3325 0    50   Input ~ 0
+SVCC
+Wire Wire Line
+	6675 3325 6775 3325
+Wire Wire Line
+	6775 3325 6775 3475
+Wire Wire Line
+	6775 3750 6775 3675
+Text GLabel 6650 3750 0    50   Input ~ 0
+SS
+Wire Wire Line
+	6650 3750 6775 3750
 $EndSCHEMATC
