File: pcb/sp0256al2/psion-speech-sp0256al2/psion-speech-sp0256al2.sch (KiCad schematic (older format))
At the start: 29 parts, among them J1 Connector_USB_B_Micro, J2 Conn_01x02_Female, J3 Conn_02x08_Odd_Even, U1 SP0256AL2, U2 74LS368, U3 PAM8302AAD, U4 74HCT00, Y1 3.2768MHz

Commit message: Updates
Parts:
- U2, U4: footprint (none) -> Package_SO:SOIC-14_3.9x8.7mm_P1.27mm
- U3: footprint (none) -> Package_SO:SO-8_5.3x6.2mm_P1.27mm
Changed lines of the file:
@@
 F 0 "U3" H 7350 2350 50  0000 C CNN
 F 1 "PAM8302AAD" H 7525 2275 50  0000 C CNN
-F 2 "" H 7800 1775 50  0001 C CNN
+F 2 "Package_SO:SO-8_5.3x6.2mm_P1.27mm" H 7800 1775 50  0001 C CNN
 F 3 "https://www.diodes.com/assets/Datasheets/PAM8302A.pdf" H 7800 1775 50  0001 C CNN
 	1    7800 1775
@@
 F 0 "U2" H 6450 4616 50  0000 C CNN
 F 1 "74LS368" H 6450 4525 50  0000 C CNN
-F 2 "" H 6450 4050 50  0001 C CNN
+F 2 "Package_SO:SOIC-14_3.9x8.7mm_P1.27mm" H 6450 4050 50  0001 C CNN
 F 3 "" H 6450 4050 50  0001 C CNN
 	1    6450 4050
@@
 F 0 "U4" H 10125 3200 50  0000 C CNN
 F 1 "74HCT00" H 10125 3109 50  0000 C CNN
-F 2 "" H 10125 2875 50  0001 C CNN
+F 2 "Package_SO:SOIC-14_3.9x8.7mm_P1.27mm" H 10125 2875 50  0001 C CNN
 F 3 "http://www.ti.com/lit/gpn/sn74hct00" H 10125 2875 50  0001 C CNN
 	1    10125 2875
@@
 F 0 "U4" H 10125 3800 50  0000 C CNN
 F 1 "74HCT00" H 10125 3709 50  0000 C CNN
-F 2 "" H 10125 3475 50  0001 C CNN
+F 2 "Package_SO:SOIC-14_3.9x8.7mm_P1.27mm" H 10125 3475 50  0001 C CNN
 F 3 "http://www.ti.com/lit/gpn/sn74hct00" H 10125 3475 50  0001 C CNN
 	2    10125 3475
@@
 F 0 "U4" H 10150 4400 50  0000 C CNN
 F 1 "74HCT00" H 10150 4309 50  0000 C CNN
-F 2 "" H 10150 4075 50  0001 C CNN
+F 2 "Package_SO:SOIC-14_3.9x8.7mm_P1.27mm" H 10150 4075 50  0001 C CNN
 F 3 "http://www.ti.com/lit/gpn/sn74hct00" H 10150 4075 50  0001 C CNN
 	3    10150 4075
@@
 F 0 "U4" H 10175 5050 50  0000 C CNN
 F 1 "74HCT00" H 10175 4959 50  0000 C CNN
-F 2 "" H 10175 4725 50  0001 C CNN
+F 2 "Package_SO:SOIC-14_3.9x8.7mm_P1.27mm" H 10175 4725 50  0001 C CNN
 F 3 "http://www.ti.com/lit/gpn/sn74hct00" H 10175 4725 50  0001 C CNN
 	4    10175 4725
@@
 F 0 "U4" H 10430 5871 50  0000 L CNN
 F 1 "74HCT00" H 10430 5780 50  0000 L CNN
-F 2 "" H 10200 5825 50  0001 C CNN
+F 2 "Package_SO:SOIC-14_3.9x8.7mm_P1.27mm" H 10200 5825 50  0001 C CNN
 F 3 "http://www.ti.com/lit/gpn/sn74hct00" H 10200 5825 50  0001 C CNN
 	5    10200 5825

Commit message: Updates
Parts:
- removed U4: 74HCT00, Package_SO:SOIC-14_3.9x8.7mm_P1.27mm, symbol 74xx:74HCT00
- added U4: 4011, Package_SO:SOIC-14_3.9x8.7mm_P1.27mm, symbol 4xxx:4011
Changed lines of the file:
@@
 Text GLabel 7000 4150 2    50   Input ~ 0
 N_SOE
-$Comp
-L 74xx:74HCT00 U4
-U 1 1 63432283
-P 10125 2875
-F 0 "U4" H 10125 3200 50  0000 C CNN
-F 1 "74HCT00" H 10125 3109 50  0000 C CNN
-F 2 "Package_SO:SOIC-14_3.9x8.7mm_P1.27mm" H 10125 2875 50  0001 C CNN
-F 3 "http://www.ti.com/lit/gpn/sn74hct00" H 10125 2875 50  0001 C CNN
-	1    10125 2875
-	1    0    0    -1
-$EndComp
-$Comp
-L 74xx:74HCT00 U4
-U 2 1 63433A3D
-P 10125 3475
-F 0 "U4" H 10125 3800 50  0000 C CNN
-F 1 "74HCT00" H 10125 3709 50  0000 C CNN
-F 2 "Package_SO:SOIC-14_3.9x8.7mm_P1.27mm" H 10125 3475 50  0001 C CNN
-F 3 "http://www.ti.com/lit/gpn/sn74hct00" H 10125 3475 50  0001 C CNN
-	2    10125 3475
-	1    0    0    -1
-$EndComp
-$Comp
-L 74xx:74HCT00 U4
-U 3 1 63434B77
-P 10150 4075
-F 0 "U4" H 10150 4400 50  0000 C CNN
-F 1 "74HCT00" H 10150 4309 50  0000 C CNN
-F 2 "Package_SO:SOIC-14_3.9x8.7mm_P1.27mm" H 10150 4075 50  0001 C CNN
-F 3 "http://www.ti.com/lit/gpn/sn74hct00" H 10150 4075 50  0001 C CNN
-	3    10150 4075
-	1    0    0    -1
-$EndComp
-$Comp
-L 74xx:74HCT00 U4
-U 4 1 63435E9B
-P 10175 4725
-F 0 "U4" H 10175 5050 50  0000 C CNN
-F 1 "74HCT00" H 10175 4959 50  0000 C CNN
-F 2 "Package_SO:SOIC-14_3.9x8.7mm_P1.27mm" H 10175 4725 50  0001 C CNN
-F 3 "http://www.ti.com/lit/gpn/sn74hct00" H 10175 4725 50  0001 C CNN
-	4    10175 4725
-	1    0    0    -1
-$EndComp
-$Comp
-L 74xx:74HCT00 U4
-U 5 1 63437A02
-P 10200 5825
-F 0 "U4" H 10430 5871 50  0000 L CNN
-F 1 "74HCT00" H 10430 5780 50  0000 L CNN
-F 2 "Package_SO:SOIC-14_3.9x8.7mm_P1.27mm" H 10200 5825 50  0001 C CNN
-F 3 "http://www.ti.com/lit/gpn/sn74hct00" H 10200 5825 50  0001 C CNN
-	5    10200 5825
-	1    0    0    -1
-$EndComp
 Text GLabel 10350 5200 2    50   Input ~ 0
 SVCC
@@
 Text GLabel 1550 4550 0    50   Input ~ 0
 VB
+$Comp
+L 4xxx:4011 U4
+U 1 1 634116DB
+P 10125 2875
+F 0 "U4" H 10125 3200 50  0000 C CNN
+F 1 "4011" H 10125 3109 50  0000 C CNN
+F 2 "Package_SO:SOIC-14_3.9x8.7mm_P1.27mm" H 10125 2875 50  0001 C CNN
+F 3 "http://www.intersil.com/content/dam/Intersil/documents/cd40/cd4011bms-12bms-23bms.pdf" H 10125 2875 50  0001 C CNN
+	1    10125 2875
+	1    0    0    -1
+$EndComp
+$Comp
+L 4xxx:4011 U4
+U 2 1 634133AD
+P 10125 3475
+F 0 "U4" H 10125 3800 50  0000 C CNN
+F 1 "4011" H 10125 3709 50  0000 C CNN
+F 2 "Package_SO:SOIC-14_3.9x8.7mm_P1.27mm" H 10125 3475 50  0001 C CNN
+F 3 "http://www.intersil.com/content/dam/Intersil/documents/cd40/cd4011bms-12bms-23bms.pdf" H 10125 3475 50  0001 C CNN
+	2    10125 3475
+	1    0    0    -1
+$EndComp
+$Comp
+L 4xxx:4011 U4
+U 3 1 63414DD2
+P 10150 4075
+F 0 "U4" H 10150 4400 50  0000 C CNN
+F 1 "4011" H 10150 4309 50  0000 C CNN
+F 2 "Package_SO:SOIC-14_3.9x8.7mm_P1.27mm" H 10150 4075 50  0001 C CNN
+F 3 "http://www.intersil.com/content/dam/Intersil/documents/cd40/cd4011bms-12bms-23bms.pdf" H 10150 4075 50  0001 C CNN
+	3    10150 4075
+	1    0    0    -1
+$EndComp
+$Comp
+L 4xxx:4011 U4
+U 4 1 63417BD8
+P 10175 4725
+F 0 "U4" H 10175 5050 50  0000 C CNN
+F 1 "4011" H 10175 4959 50  0000 C CNN
+F 2 "Package_SO:SOIC-14_3.9x8.7mm_P1.27mm" H 10175 4725 50  0001 C CNN
+F 3 "http://www.intersil.com/content/dam/Intersil/documents/cd40/cd4011bms-12bms-23bms.pdf" H 10175 4725 50  0001 C CNN
+	4    10175 4725
+	1    0    0    -1
+$EndComp
+$Comp
+L 4xxx:4011 U4
+U 5 1 63419811
+P 10200 5825
+F 0 "U4" H 10430 5871 50  0000 L CNN
+F 1 "4011" H 10430 5780 50  0000 L CNN
+F 2 "Package_SO:SOIC-14_3.9x8.7mm_P1.27mm" H 10200 5825 50  0001 C CNN
+F 3 "http://www.intersil.com/content/dam/Intersil/documents/cd40/cd4011bms-12bms-23bms.pdf" H 10200 5825 50  0001 C CNN
+	5    10200 5825
+	1    0    0    -1
+$EndComp
 $EndSCHEMATC

Commit message: Updates
Parts:
- removed J2: Conn_01x02_Female, Connector_PinHeader_2.54mm:PinHeader_1x02_P2.54mm_Vertical, symbol Connector:Conn_01x02_Female
- added LS1: Speaker, symbol Device:Speaker
Connections:
- net at C9.1, FB2.1: now also LS1.1
- net at C8.1, FB3.1: now also LS1.2
Other:
- note added: "PB mounted speaker can be a\nwired sounder of\nsome other type."
Changed lines of the file:
@@
 Wire Wire Line
 	8850 1775 8850 1850
-$Comp
-L Connector:Conn_01x02_Female J2
-U 1 1 6342C3EE
-P 9850 1575
-F 0 "J2" H 9878 1551 50  0000 L CNN
-F 1 "Conn_01x02_Female" H 9878 1460 50  0000 L CNN
-F 2 "Connector_PinHeader_2.54mm:PinHeader_1x02_P2.54mm_Vertical" H 9850 1575 50  0001 C CNN
-F 3 "~" H 9850 1575 50  0001 C CNN
-	1    9850 1575
-	1    0    0    -1
-$EndComp
 Wire Wire Line
 	9650 1575 9375 1575
@@
 	1    0    0    -1
 $EndComp
+$Comp
+L Device:Speaker LS1
+U 1 1 63412366
+P 9850 1575
+F 0 "LS1" H 10020 1571 50  0000 L CNN
+F 1 "Speaker" H 10020 1480 50  0000 L CNN
+F 2 "" H 9850 1375 50  0001 C CNN
+F 3 "~" H 9840 1525 50  0001 C CNN
+	1    9850 1575
+	1    0    0    -1
+$EndComp
+Text Notes 9900 2100 0    50   ~ 0
+PB mounted speaker can be a\nwired sounder of\nsome other type.
 $EndSCHEMATC

Commit message: Updates
Parts:
- removed LS1: Speaker, symbol Device:Speaker
- added J2: AudioJack2_Ground_Switch, symbol Connector:AudioJack2_Ground_Switch
- added J4: Conn_01x02_Female, Connector_PinHeader_2.54mm:PinHeader_1x02_P2.54mm_Vertical, symbol Connector:Conn_01x02_Female
- Y1: footprint (none) -> psion_org_2:crystal_um4s
Connections:
- net at C9.1, FB2.1: now also J4.1 (Pin_1)
- net at C8.1, FB3.1: now also J4.2 (Pin_2)
- net at C5.1, R2.1: now also J2.S, J2.T; no longer R3.1
- new net: J2.SN, R3.1
Other:
- moved on the sheet: C11
Changed lines of the file:
@@
 F 0 "Y1" V 4254 1756 50  0000 L CNN
 F 1 "3.2768MHz" V 4345 1756 50  0000 L CNN
-F 2 "" H 4300 1625 50  0001 C CNN
+F 2 "psion_org_2:crystal_um4s" H 4300 1625 50  0001 C CNN
 F 3 "~" H 4300 1625 50  0001 C CNN
 	1    4300 1625
@@
 AR Path="/63427936" Ref="FB2"  Part="1"
 F 0 "FB2" V 8375 1575 50  0000 C CNN
-F 1 "Laird Technologies Part # MI0805K400R-10" V 8025 2300 50  0000 C CNN
+F 1 "Laird Technologies Part # MI0805K400R-10" V 7600 1325 50  0000 C CNN
 F 2 "Capacitor_SMD:C_0805_2012Metric" V 8455 1575 50  0001 C CNN
 F 3 "~" H 8525 1575 50  0001 C CNN
@@
 Wire Wire Line
 	8850 1775 8850 1850
-Wire Wire Line
-	9650 1575 9375 1575
 Connection ~ 9375 1575
-Wire Wire Line
-	9650 1675 9650 1775
-Wire Wire Line
-	9650 1775 8850 1775
 Wire Wire Line
 	9375 1575 9375 1850
@@
 Wire Wire Line
 	6125 1325 6125 1425
-Wire Wire Line
-	4875 2550 5375 2550
-Wire Wire Line
-	5375 2550 5375 750
-Wire Wire Line
-	5375 750  6125 750
 Wire Wire Line
 	6125 750  6125 1125
@@
 L Device:C_Small C11
 U 1 1 6348419A
-P 10650 1200
-F 0 "C11" H 10742 1246 50  0000 L CNN
-F 1 "10uF" H 10742 1155 50  0000 L CNN
-F 2 "Capacitor_SMD:C_1210_3225Metric_Pad1.33x2.70mm_HandSolder" H 10650 1200 50  0001 C CNN
-F 3 "~" H 10650 1200 50  0001 C CNN
-	1    10650 1200
+P 6950 2575
+F 0 "C11" H 7042 2621 50  0000 L CNN
+F 1 "10uF" H 7042 2530 50  0000 L CNN
+F 2 "Capacitor_SMD:C_1210_3225Metric_Pad1.33x2.70mm_HandSolder" H 6950 2575 50  0001 C CNN
+F 3 "~" H 6950 2575 50  0001 C CNN
+	1    6950 2575
 	1    0    0    -1
 $EndComp
@@
 L power:GND #PWR014
 U 1 1 63484BC1
-P 10650 1425
-F 0 "#PWR014" H 10650 1175 50  0001 C CNN
-F 1 "GND" H 10655 1252 50  0000 C CNN
-F 2 "" H 10650 1425 50  0001 C CNN
-F 3 "" H 10650 1425 50  0001 C CNN
-	1    10650 1425
-	1    0    0    -1
-$EndComp
-Text GLabel 10600 925  0    50   Input ~ 0
+P 6950 2800
+F 0 "#PWR014" H 6950 2550 50  0001 C CNN
+F 1 "GND" H 6955 2627 50  0000 C CNN
+F 2 "" H 6950 2800 50  0001 C CNN
+F 3 "" H 6950 2800 50  0001 C CNN
+	1    6950 2800
+	1    0    0    -1
+$EndComp
+Text GLabel 6900 2300 0    50   Input ~ 0
 SVCC
 Wire Wire Line
-	10600 925  10650 925
-Wire Wire Line
-	10650 925  10650 1100
-Wire Wire Line
-	10650 1300 10650 1425
+	6900 2300 6950 2300
+Wire Wire Line
+	6950 2300 6950 2475
+Wire Wire Line
+	6950 2675 6950 2800
 Text GLabel 2050 4150 2    50   Input ~ 0
 SD1
@@
 	1    0    0    -1
 $EndComp
-$Comp
-L Device:Speaker LS1
-U 1 1 63412366
-P 9850 1575
-F 0 "LS1" H 10020 1571 50  0000 L CNN
-F 1 "Speaker" H 10020 1480 50  0000 L CNN
-F 2 "" H 9850 1375 50  0001 C CNN
-F 3 "~" H 9840 1525 50  0001 C CNN
-	1    9850 1575
-	1    0    0    -1
-$EndComp
-Text Notes 9900 2100 0    50   ~ 0
+Text Notes 7950 1050 0    50   ~ 0
 PB mounted speaker can be a\nwired sounder of\nsome other type.
+$Comp
+L Connector:AudioJack2_Ground_Switch J2
+U 1 1 6343E58B
+P 5750 2550
+F 0 "J2" H 5570 2568 50  0000 R CNN
+F 1 "AudioJack2_Ground_Switch" H 5570 2477 50  0000 R CNN
+F 2 "" H 5750 2750 50  0001 C CNN
+F 3 "~" H 5750 2750 50  0001 C CNN
+	1    5750 2550
+	-1   0    0    -1
+$EndComp
+Wire Wire Line
+	9375 1575 9850 1575
+Wire Wire Line
+	9850 1675 9750 1675
+Wire Wire Line
+	9750 1675 9750 1775
+Wire Wire Line
+	8850 1775 9750 1775
+Wire Wire Line
+	4875 2550 5325 2550
+Wire Wire Line
+	5325 2550 5325 2350
+Wire Wire Line
+	5325 2350 5550 2350
+Connection ~ 5325 2550
+Wire Wire Line
+	5325 2550 5550 2550
+Wire Wire Line
+	5250 2450 5250 750
+Wire Wire Line
+	5250 750  6125 750
+Wire Wire Line
+	5250 2450 5550 2450
+$Comp
+L Connector:Conn_01x02_Female J4
+U 1 1 634738A3
+P 10050 1575
+F 0 "J4" H 10078 1551 50  0000 L CNN
+F 1 "Conn_01x02_Female" H 10078 1460 50  0000 L CNN
+F 2 "Connector_PinHeader_2.54mm:PinHeader_1x02_P2.54mm_Vertical" H 10050 1575 50  0001 C CNN
+F 3 "~" H 10050 1575 50  0001 C CNN
+	1    10050 1575
+	1    0    0    -1
+$EndComp
 $EndSCHEMATC

Commit message: Updates
Parts:
- J2: footprint (none) -> psion_org_2:truconnect_stereo_audio_5_pin
- RV1: footprint Resistor_SMD:R_0805_2012Metric -> Potentiometer_THT:Potentiometer_Bourns_3296W_Vertical
Connections:
- net GND: now also J2.G
Changed lines of the file:
@@
 F 0 "RV1" H 6056 1621 50  0000 R CNN
 F 1 "10k" H 6056 1530 50  0000 R CNN
-F 2 "Resistor_SMD:R_0805_2012Metric" H 6125 1575 50  0001 C CNN
+F 2 "Potentiometer_THT:Potentiometer_Bourns_3296W_Vertical" H 6125 1575 50  0001 C CNN
 F 3 "~" H 6125 1575 50  0001 C CNN
 	1    6125 1575
@@
 F 0 "J2" H 5570 2568 50  0000 R CNN
 F 1 "AudioJack2_Ground_Switch" H 5570 2477 50  0000 R CNN
-F 2 "" H 5750 2750 50  0001 C CNN
+F 2 "psion_org_2:truconnect_stereo_audio_5_pin" H 5750 2750 50  0001 C CNN
 F 3 "~" H 5750 2750 50  0001 C CNN
 	1    5750 2550
@@
 	1    0    0    -1
 $EndComp
+$Comp
+L power:GND #PWR0102
+U 1 1 6348B625
+P 5750 2850
+F 0 "#PWR0102" H 5750 2600 50  0001 C CNN
+F 1 "GND" H 5755 2677 50  0000 C CNN
+F 2 "" H 5750 2850 50  0001 C CNN
+F 3 "" H 5750 2850 50  0001 C CNN
+	1    5750 2850
+	1    0    0    -1
+$EndComp

Commit message: Updates
Parts:
- removed U2: 74LS368, Package_SO:SOIC-14_3.9x8.7mm_P1.27mm, symbol 74xx_IEEE:74LS368
- added U5: 74LS368, Package_SO:SOIC-16_3.9x9.9mm_P1.27mm, symbol 74xx:74LS368
Connections:
- net GND: now also U5.8 (GND)
- net LRQ: now also U5.14 (I6)
- net NOT_SEL_SOE_1: now also U5.9 (O4a)
- net N_SOE: now also U5.7 (O3a)
- net N_SS: now also U5.3 (O1a)
- net SD7: now also U5.11 (O5b)
- net SEL_SOE_1: now also U5.10 (I4), U5.15 (OEb)
- net SOE: now also U5.6 (I3)
- net SS: now also U5.2 (I1)
- net SVCC: now also U5.16 (VCC); no longer C10.1, U4.14 (VDD)
- new net: C10.1, U4.14 (VDD)
- new net: U5.12 (I5), U5.13 (O6b)
Changed lines of the file:
@@
 	2225 5350 2225 6225
 $Sheet
-S 5450 5700 1200 625
+S 3625 5250 1200 625
 U 6340FD7B
 F0 "Psion ROM" 50
@@
 Text GLabel 1875 2875 0    50   Input ~ 0
 SD5
-$Comp
-L 74xx_IEEE:74LS368 U2
-U 1 1 63421380
-P 6450 4050
-F 0 "U2" H 6450 4616 50  0000 C CNN
-F 1 "74LS368" H 6450 4525 50  0000 C CNN
-F 2 "Package_SO:SOIC-14_3.9x8.7mm_P1.27mm" H 6450 4050 50  0001 C CNN
-F 3 "" H 6450 4050 50  0001 C CNN
-	1    6450 4050
-	1    0    0    -1
-$EndComp
-Text GLabel 7000 4650 2    50   Input ~ 0
+Text GLabel 8450 5225 2    50   Input ~ 0
 SD7
-Wire Wire Line
-	5900 4650 5625 4650
-Wire Wire Line
-	5625 4650 5625 4950
-Wire Wire Line
-	5625 4950 7000 4950
-Wire Wire Line
-	7000 4950 7000 4750
-Text GLabel 5900 4750 0    50   Input ~ 0
+Text GLabel 7450 5325 0    50   Input ~ 0
 LRQ
-$Comp
-L power:GND #PWR08
-U 1 1 634277F0
-P 5400 3800
-F 0 "#PWR08" H 5400 3550 50  0001 C CNN
-F 1 "GND" H 5405 3627 50  0000 C CNN
-F 2 "" H 5400 3800 50  0001 C CNN
-F 3 "" H 5400 3800 50  0001 C CNN
-	1    5400 3800
-	-1   0    0    -1
-$EndComp
-Wire Wire Line
-	5900 3800 5400 3800
-Text GLabel 5900 3950 0    50   Input ~ 0
+Text GLabel 7450 4825 0    50   Input ~ 0
 SS
-Text GLabel 5900 4150 0    50   Input ~ 0
+Text GLabel 7450 5025 0    50   Input ~ 0
 SOE
-Text GLabel 7000 3950 2    50   Input ~ 0
+Text GLabel 8450 4825 2    50   Input ~ 0
 N_SS
-Text GLabel 7000 4150 2    50   Input ~ 0
+Text GLabel 8450 5025 2    50   Input ~ 0
 N_SOE
-Text GLabel 10350 5200 2    50   Input ~ 0
+Text GLabel 8100 4150 2    50   Input ~ 0
 SVCC
 Wire Wire Line
@@
 Wire Wire Line
 	9575 4825 9875 4825
-Text GLabel 5900 4250 0    50   Input ~ 0
+Text GLabel 6850 5125 0    50   Input ~ 0
 SEL_SOE_1
-Text GLabel 7000 4250 2    50   Input ~ 0
+Text GLabel 8450 5125 2    50   Input ~ 0
 NOT_SEL_SOE_1
 Text GLabel 10475 4725 2    50   Input ~ 0
@@
 	1    0    0    -1
 $EndComp
+$Comp
+L 74xx:74LS368 U5
+U 1 1 6360F2CE
+P 7950 5225
+F 0 "U5" H 8250 6100 50  0000 C CNN
+F 1 "74LS368" H 8375 6025 50  0000 C CNN
+F 2 "Package_SO:SOIC-16_3.9x9.9mm_P1.27mm" H 7950 5225 50  0001 C CNN
+F 3 "http://www.ti.com/lit/gpn/sn74LS368" H 7950 5225 50  0001 C CNN
+	1    7950 5225
+	1    0    0    -1
+$EndComp
+Wire Wire Line
+	8450 5325 8725 5325
+Wire Wire Line
+	8725 5325 8725 6425
+Wire Wire Line
+	8725 6425 7050 6425
+Wire Wire Line
+	7050 6425 7050 5225
+Wire Wire Line
+	7050 5225 7450 5225
+$Comp
+L power:GND #PWR0103
+U 1 1 6361864B
+P 7950 6075
+F 0 "#PWR0103" H 7950 5825 50  0001 C CNN
+F 1 "GND" H 7955 5902 50  0000 C CNN
+F 2 "" H 7950 6075 50  0001 C CNN
+F 3 "" H 7950 6075 50  0001 C CNN
+	1    7950 6075
+	1    0    0    -1
+$EndComp
+Wire Wire Line
+	7950 6075 7950 5925
+Wire Wire Line
+	7950 4150 8100 4150
+Wire Wire Line
+	7950 4150 7950 4525
+Wire Wire Line
+	7450 5125 7150 5125
+Wire Wire Line
+	7150 5625 7450 5625
+Wire Wire Line
+	7150 5125 7150 5625
+Connection ~ 7150 5125
+Wire Wire Line
+	7150 5125 6850 5125
 $EndSCHEMATC

Commit message: Updates
Parts:
- added R7: 47k, Resistor_SMD:R_0805_2012Metric, symbol Device:R_Small
Connections:
- net GND: now also U1.22 (TEST), U5.1 (OEa), R7.2
- net SVCC: now also C10.1, U4.14 (VDD), R7.1; no longer U1.22 (TEST)
Other:
- note added: "SEL_SOE_0 SS=0 SOE=0\nSEL_SOE_1 SS=0 SOE=1"
Changed lines of the file:
@@
 Connection ~ 1575 2575
 Wire Wire Line
-	1575 3225 1575 2675
+	1575 3225 1575 3150
 Connection ~ 1575 2675
 Text GLabel 3475 2575 2    50   Input ~ 0
@@
 Wire Wire Line
 	3175 2575 3425 2575
-Wire Wire Line
-	3425 2575 3425 2275
-Wire Wire Line
-	3425 2275 3175 2275
 Connection ~ 3425 2575
 Wire Wire Line
 	3425 2575 3475 2575
 Wire Wire Line
-	3425 2275 3425 2175
-Wire Wire Line
 	3425 2175 3175 2175
-Connection ~ 3425 2275
 $Comp
 L Device:C_Small C10
@@
 $EndComp
 Wire Wire Line
-	7950 6075 7950 5925
+	7950 6075 7950 5975
 Wire Wire Line
 	7950 4150 8100 4150
@@
 Wire Wire Line
 	7150 5125 6850 5125
+Wire Wire Line
+	7950 5975 7300 5975
+Wire Wire Line
+	7300 5975 7300 5525
+Wire Wire Line
+	7300 5525 7450 5525
+Connection ~ 7950 5975
+Wire Wire Line
+	7950 5975 7950 5925
+Wire Wire Line
+	3425 2175 3425 2575
+Wire Wire Line
+	3175 2275 3875 2275
+Wire Wire Line
+	3875 2275 3875 3150
+Wire Wire Line
+	3875 3150 1575 3150
+Connection ~ 1575 3150
+Wire Wire Line
+	1575 3150 1575 2675
+Text Notes 7375 3225 0    50   ~ 0
+SEL_SOE_0          SS=0   SOE=0\nSEL_SOE_1          SS=0   SOE=1
+Text GLabel 10350 5200 2    50   Input ~ 0
+SVCC
+$Comp
+L Device:R_Small R7
+U 1 1 6369783E
+P 5475 4150
+F 0 "R7" H 5534 4196 50  0000 L CNN
+F 1 "47k" H 5534 4105 50  0000 L CNN
+F 2 "Resistor_SMD:R_0805_2012Metric" H 5475 4150 50  0001 C CNN
+F 3 "~" H 5475 4150 50  0001 C CNN
+	1    5475 4150
+	1    0    0    -1
+$EndComp
+Text GLabel 5575 3775 2    50   Input ~ 0
+SVCC
+Wire Wire Line
+	5475 4050 5475 3775
+Wire Wire Line
+	5475 3775 5575 3775
+$Comp
+L power:GND #PWR0104
+U 1 1 636A0972
+P 5475 4425
+F 0 "#PWR0104" H 5475 4175 50  0001 C CNN
+F 1 "GND" H 5480 4252 50  0000 C CNN
+F 2 "" H 5475 4425 50  0001 C CNN
+F 3 "" H 5475 4425 50  0001 C CNN
+	1    5475 4425
+	1    0    0    -1
+$EndComp
+Wire Wire Line
+	5475 4425 5475 4250
 $EndSCHEMATC
