File: pcb/sp0256al2/psion-speech-sp0256al2/psion-speech-sp0256al2.sch (KiCad schematic (older format))
At the start: 38 parts, among them J1 Connector_USB_B_Micro, J2 AudioJack2_Ground_Switch, J3 Conn_02x08_Odd_Even, J4 Conn_01x02_Female, U1 SP0256AL2, U3 PAM8302AAD, U4 4011, U5 74LS368, Y1 3.2768MHz

Commit message: Updates
Parts:
- C8, C9: value 220pF -> 100nF
Other:
- note added: "PCB mounted speaker can be a\nwired sounder or\nsome other type."
- note removed: "PB mounted speaker can be a\nwired sounder of\nsome other type."
Changed lines of the file:
@@
 P 8850 1950
 F 0 "C8" H 8942 1996 50  0000 L CNN
-F 1 "220pF" H 8942 1905 50  0000 L CNN
+F 1 "100nF" H 8942 1905 50  0000 L CNN
 F 2 "Capacitor_SMD:C_0805_2012Metric" H 8850 1950 50  0001 C CNN
 F 3 "~" H 8850 1950 50  0001 C CNN
@@
 P 9375 1950
 F 0 "C9" H 9467 1996 50  0000 L CNN
-F 1 "220pF" H 9467 1905 50  0000 L CNN
+F 1 "100nF" H 9467 1905 50  0000 L CNN
 F 2 "Capacitor_SMD:C_0805_2012Metric" H 9375 1950 50  0001 C CNN
 F 3 "~" H 9375 1950 50  0001 C CNN
@@
 $EndComp
 Text Notes 9975 1150 0    50   ~ 0
-PB mounted speaker can be a\nwired sounder of\nsome other type.
+PCB mounted speaker can be a\nwired sounder or\nsome other type.
 $Comp
 L Connector:AudioJack2_Ground_Switch J2
